File: 18 processor.65265/mapper.kicad_sch (KiCad schematic)
At the start: 24 parts, among them Q1 2N3906, Q2 2N3906, U12 74LS688, U18 PCF8584, U20 GAL22V10, U25 74LS374, U4 74LS07, U7 74LS04

Commit message: 02 and 265
Parts:
- SP1, SP2: footprint Jameco PCB Speaker 30mm 135722:Jameco PCB Speaker 30mm 135722 -> CUSTOM:JAMECO SPEAKER
Changed lines of the file:
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@@
     (property "Reference" "SP2" (id 0) (at 371.1702 82.1182 0))
     (property "Value" "SPEAKER" (id 1) (at 371.1702 84.4296 0))
-    (property "Footprint" "Jameco PCB Speaker 30mm 135722:Jameco PCB Speaker 30mm 135722" (id 2) (at 372.11 87.63 0)
+    (property "Footprint" "CUSTOM:JAMECO SPEAKER" (id 2) (at 372.11 87.63 0)
       (effects (font (size 1.27 1.27)) hide)
     )
@@
     (property "Reference" "SP1" (id 0) (at 367.9952 45.9232 0))
     (property "Value" "SPEAKER" (id 1) (at 367.9952 48.2346 0))
-    (property "Footprint" "Jameco PCB Speaker 30mm 135722:Jameco PCB Speaker 30mm 135722" (id 2) (at 368.935 51.435 0)
-      (effects (font (size 1.27 1.27)) hide)
-    )
+    (property "Footprint" "CUSTOM:JAMECO SPEAKER" (id 2) (at 368.935 51.435 0)
+      (effects (font (size 1.27 1.27)) hide)
+    )
