File: 18 processor.65265/power.kicad_sch (KiCad schematic)
At the start: 53 parts, among them U16 74LS08, U17 74LS00, U21 74LS74, U26 74LS32, U3 74LS14, U4 74LS07, U7 74LS04

Commit message: 02 and 265
Parts:
- removed U16: 74LS08, Package_DIP:DIP-14_W7.62mm_Socket_LongPads, symbol 74xx:74LS08
Connections:
- no-connect marks 45 -> 33
Other:
- moved on the sheet: U3D, U3E, U4D
