File: 18 processor.65265/processor.65816.kicad_pcb (KiCad board)
At the start: 2 copper layers, 235 x 160 mm, 117 parts, among them J1 IO Address Select, J11 FPANEL, J2 65816 RESET, J3 65816 ONLY, P1 CONN_02X25, P2 CONN_02X25, P3 CONN_02X25, Q1 2N3906, Q2 2N3906, SW1 RESET, U1 74LS244, U10 GAL16V8, U11 74LS244, U12 74LS688, U13 CPU CLOCK, U14 W65C265SxPL, U15 DS1233, U17 74LS00, U18 PCF8584, U19 27C64, U2 UART CLOCK, U20 GAL22V10, U21 74LS74, U22 74LS688, U23 74LS244, U25 74LS374, U26 74LS32, U3 74LS14, U31 74LS244, U33 74LS374, U4 74LS07, U5 74LS244, U6 74LS244, U7 74LS04, U8 74LS245, U9 GAL22V10

Commit message: duodyne 6502 work
Parts:
- moved U19 10.3 mm to (91.0, 122.6)
Routing:
- net GND: track 0.00 -> 1583.9 mm
- net VCC: track 0.00 -> 1375.8 mm, vias 0 -> 1
- net ~{RES_OUT}: track 0.00 -> 409.4 mm, vias 0 -> 1
- net I2C_SDA: track 0.00 -> 403.5 mm, vias 0 -> 2
- net CPU-D1: track 0.00 -> 369.6 mm, vias 0 -> 6
- net CPU-D6: track 0.00 -> 367.9 mm, vias 0 -> 1
- net ~{65816EN}: track 0.00 -> 361.7 mm, vias 0 -> 2
- net CPU-D0: track 0.00 -> 356.8 mm, vias 0 -> 7
- net CPU-D3: track 0.00 -> 352.9 mm, vias 0 -> 2
- net CPU-D5: track 0.00 -> 344.6 mm, vias 0 -> 6
- net I2C_SCL: track 0.00 -> 343.5 mm, vias 0 -> 4
- net CPU-D4: track 0.00 -> 337.0 mm, vias 0 -> 1
- net CPU-D2: track 0.00 -> 322.8 mm, vias 0 -> 8
- net CPU-D7: track 0.00 -> 291.7 mm, vias 0 -> 3
- net ~{EXT_RES}: track 0.00 -> 284.8 mm, vias 0 -> 2
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- added copper zone on B.Cu, net GND
- added copper zone on F.Cu, net GND
