File: 13 front-panel.processor ALT/hardware/front-panel.processor.kicad_pcb (KiCad board)
At the start: 2 copper layers, 295 x 80 mm, 40 parts, among them J1 FPANEL, J2 TTL SERIAL, J3 MICRO SD CARD, J4 TTL Serial to WiFi Enable, J5 Micro_SD_Card, SW1 SW_SPDT, SW10 SW_SPDT, SW11 SW_SPDT, SW12 SW_SPDT, SW2 SW_SPDT, SW3 SW_SPDT, SW4 SW_SPDT, SW5 SW_SPDT, SW6 SW_SPDT, SW7 SW_SPDT, SW8 SW_SPDT, SW9 SW_Push, U1 74LS240, U2 ESP32-S3-DevKitC, U5 LP2950-3.3_TO92

Commit message: duodyne 6502 work
Parts:
- added C3: 0.1u, Capacitor_THT:C_Disc_D5.0mm_W2.5mm_P5.00mm, F.Cu at (198.8, 166.3)
- added D10: GRN-SD R/W+RED-ERR, LED_THT:LED_D5.0mm, F.Cu at (224.7, 156.0)
- added J6: UPDI ONLY, Connector_PinHeader_2.54mm:PinHeader_1x06_P2.54mm_Vertical, F.Cu at (285.0, 227.2)
- added R3: 10K, Resistor_THT:R_Axial_DIN0207_L6.3mm_D2.5mm_P7.62mm_Horizontal, F.Cu at (198.8, 154.1)
- added R4: 10K, Resistor_THT:R_Axial_DIN0207_L6.3mm_D2.5mm_P7.62mm_Horizontal, F.Cu at (198.8, 158.2)
- added R5: 220, Resistor_THT:R_Axial_DIN0207_L6.3mm_D2.5mm_P7.62mm_Horizontal, F.Cu at (198.8, 162.2)
- added R7: 4700, Resistor_THT:R_Axial_DIN0207_L6.3mm_D2.5mm_P7.62mm_Horizontal, F.Cu at (309.5, 227.0)
- added U7: ATtiny1614-SS, Package_SO:SOIC-14_3.9x8.7mm_P1.27mm, F.Cu at (267.9, 221.4)
Connections:
- U2 pad 27: LV_I2C_SCL -> IC_RX
- U2 pad 32: LV_I2C_SDA -> IC_TX
Routing:
- net VCC: track 583.9 -> 352.4 mm, vias 8 -> 1
- net Net-(U7-PB2): track 0.00 -> 132.6 mm, vias 0 -> 1
- net GND: track 893.3 -> 791.5 mm, vias 8 -> 0
- net Net-(D10-KA): track 0.00 -> 85.1 mm, vias 0 -> 3
- net /LED5: track 119.8 -> 53.7 mm, vias 3 -> 1
- net DI: track 262.4 -> 319.1 mm, vias 1 -> 0
- net LV_I2C_SDA: track 76.9 -> 131.7 mm, vias 0 -> 1
- net IC_TX: track 0.00 -> 52.0 mm
- net /LED1: track 101.9 -> 51.0 mm
- net +3.3V: track 292.5 -> 342.9 mm, vias 6 -> 1
- net /LED4: track 93.8 -> 45.2 mm, vias 2 -> 1
- net /LED2: track 95.4 -> 47.8 mm, vias 6 -> 0
- net /LED0: track 98.7 -> 53.8 mm, vias 3 -> 1
- net /LED6: track 106.4 -> 63.3 mm, vias 3 -> 1
- net LV_I2C_SCL: track 92.7 -> 135.5 mm
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Other:
- board text added: "FRONT PANEL ALT, PROCESSOR, VERSION 1.1, AS OF 19 APRIL 2025"
- board text removed: "FRONT PANEL ALT, PROCESSOR, VERSION 1.1, AS OF 31 MARCH 2025"
