File: 13 front-panel.processor ALT/hardware/front-panel.processor.kicad_sch (KiCad schematic)
At the start: 40 parts, among them J1 FPANEL, J2 TTL SERIAL, J3 MICRO SD CARD, J4 TTL Serial to WiFi Enable, J5 Micro_SD_Card, SW1 SW_SPDT, SW10 SW_SPDT, SW11 SW_SPDT, SW12 SW_SPDT, SW2 SW_SPDT, SW3 SW_SPDT, SW4 SW_SPDT, SW5 SW_SPDT, SW6 SW_SPDT, SW7 SW_SPDT, SW8 SW_SPDT, SW9 SW_Push, U1 74LS240, U2 ESP32-S3-DevKitC, U5 LP2950-3.3_TO92

Commit message: duodyne 6502 work
Parts:
- added C3: 0.1u, Capacitor_THT:C_Disc_D5.0mm_W2.5mm_P5.00mm, symbol Device:C
- added D10: GRN-SD R/W+RED-ERR, LED_THT:LED_D5.0mm, symbol Device:LED_Dual_Bidirectional
- added J6: UPDI ONLY, Connector_PinHeader_2.54mm:PinHeader_1x06_P2.54mm_Vertical, symbol Connector_Generic:Conn_01x06
- added R3, R4: 10K, Resistor_THT:R_Axial_DIN0207_L6.3mm_D2.5mm_P7.62mm_Horizontal, symbol Device:R
- added R5: 220, Resistor_THT:R_Axial_DIN0207_L6.3mm_D2.5mm_P7.62mm_Horizontal, symbol Device:R
- added R7: 4700, Resistor_THT:R_Axial_DIN0207_L6.3mm_D2.5mm_P7.62mm_Horizontal, symbol Device:R
- added U7: ATtiny1614-SS, Package_SO:SOIC-14_3.9x8.7mm_P1.27mm, symbol MCU_Microchip_ATtiny:ATtiny1614-SS
Connections:
- net +3.3V: now also C3.2, J6.3 (Pin_3), R3.1, R4.1, U7.1 (VCC)
- net CLK: now also U7.13 (PA3)
- net CS: now also U7.2 (PA4)
- net DI: now also U7.11 (PA1)
- net DO: now also U7.12 (PA2)
- net GND: now also C3.1, J6.1 (Pin_1), U7.14 (GND)
- net LV_I2C_SCL: now also R3.2, U7.9 (PB0); no longer U2.27 (GPIO21)
- net LV_I2C_SDA: now also R4.2, U7.8 (PB1); no longer U2.32 (GPIO35)
- new net: R5.1, U7.7 (PB2)
- new net: D10.2 (AK), R5.2
- new net: D10.1 (KA), U7.6 (PB3)
- new net IC_RX: U2.27 (GPIO21), U7.3 (PA5)
- new net IC_TX: U2.32 (GPIO35), U7.4 (PA6)
- new net UPDI: J6.4 (Pin_4), R7.2, U7.10 (~{RESET}/PA0)
- new net UPDI-TX: J6.5 (Pin_5), R7.1
- no-connect marks 43 -> 46
Other:
- note added: "NOTE: I2C TO SD CARD CIRCUIT BASED ON http://www.technoblogy.com/show?3XEP"
- note added: "NOTE: ONLY ATTEMPT UPDI PROGRAMMING WITH FRONT PANEL DISCONNECTED FROM Z80 PROCESSOR BOARD."
- note added: "USB TO UPDI INTERFACE"
- moved on the sheet: D5, H1, H2, H3, H4, J3, J5, R6
