File: 22 processor.6502/hardware/bussharing.kicad_sch (KiCad schematic)
At the start: 13 parts, among them J1 IO Address Select, J2 6809 RESET, J3 6809 ONLY, U1 74LS04, U16 74LS08, U21 74LS74, U22 74LS688, U4 74LS07, U7 74LS14

Commit message: duodyne 6502 work
Parts:
- J2: value 6809 RESET -> 6502 RESET
- J3: value 6809 ONLY -> 6502 ONLY
Other:
- note added: "Note: IO Address Port $9F 1-2 =off - A7 (high) 3-4 =on - A6 (low) 5-6 =on - A5 (low) 7-8 =off - A4 (high) 9-10 =off - A3 (high) 11-12 =off - A2 (high) 13-14 =off - A1 (high) 15-16 =off - A0 (high)"
- note removed: "Note: IO Address Port $96 1-2 =off - A7 (high) 3-4 =on - A6 (low) 5-6 =on - A5 (low) 7-8 =off - A4 (high) 9-10 =on - A3 (low) 11-12 =off - A2 (high) 13-14 =off - A1 (high) 15-16 =on - A0 (low)"
Changed lines of the file:
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@@
   (title_block
     (title "Duodyne 6502 CPU board")
-    (date "2025-04-12")
-    (rev "V0.8")
+    (date "2025-04-26")
+    (rev "V0.9")
   )
   (junction (at 70.104 72.644) (diameter 0) (color 0 0 0 0)
@@
     (effects (font (size 1.016 1.016)) (justify left bottom))
   )
-  (text "Note: IO Address Port $96\n1-2 =off - A7 (high)\n3-4 =on - A6 (low)\n5-6 =on - A5 (low)\n7-8 =off - A4 (high)\n9-10 =on - A3 (low)\n11-12 =off - A2 (high)\n13-14 =off - A1 (high)\n15-16 =on - A0 (low)"
+  (text "Note: IO Address Port $9F\n1-2   =off - A7 (high)\n3-4   =on  - A6 (low)\n5-6   =on  - A5 (low)\n7-8   =off - A4 (high)\n9-10  =off - A3 (high)\n11-12 =off - A2 (high)\n13-14 =off - A1 (high)\n15-16 =off - A0 (high)"
     (at 27.559 46.609 0)
     (effects (font (size 1.524 1.524)) (justify left bottom))
@@
       (effects (font (size 1.27 1.27)) (justify right))
     )
-    (property "Value" "6809 ONLY" (id 1) (at 149.9362 67.2592 0)
+    (property "Value" "6502 ONLY" (id 1) (at 149.9362 67.2592 0)
       (effects (font (size 1.27 1.27)) (justify right))
     )
@@
       (effects (font (size 1.27 1.27)) (justify right))
     )
-    (property "Value" "6809 RESET" (id 1) (at 140.2588 86.4108 0)
+    (property "Value" "6502 RESET" (id 1) (at 140.2588 86.4108 0)
       (effects (font (size 1.27 1.27)) (justify right))
     )
