File: 22 processor.6502/hardware/power.kicad_sch (KiCad schematic)
At the start: 50 parts, among them U1 74LS04, U16 74LS08, U21 74LS74, U4 74LS07, U7 74LS14

Commit message: duodyne 6502 work
Parts:
- added unit 2 of U1
- added unit 2 of U7
Connections:
- no-connect marks 11 -> 15
Changed lines of the file:
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@@
   (title_block
     (title "Duodyne 6502 CPU board")
-    (date "2025-04-12")
-    (rev "V0.8")
+    (date "2025-04-26")
+    (rev "V0.9")
   )
   (junction (at 214.63 111.76) (diameter 0) (color 0 0 0 0)
@@
   (junction (at 184.15 124.46) (diameter 0) (color 0 0 0 0)
   )
+  (no_connect (at 49.53 203.835))
+  (no_connect (at 49.53 216.535))
   (no_connect (at 79.756 169.418))
   (no_connect (at 50.038 174.498))
@@
   (no_connect (at 65.278 177.038))
   (no_connect (at 87.376 174.498))
+  (no_connect (at 64.77 203.835))
   (no_connect (at 50.038 192.024))
+  (no_connect (at 64.77 216.535))
   (no_connect (at 50.038 179.578))
   (no_connect (at 72.136 179.578))
@@
     (pin "1")
   )
+  (symbol (lib_id "74xx:74LS04") (at 57.15 203.835 0) (unit 2)
+    (in_bom yes) (on_board yes)
+    (property "Reference" "U1" (id 0) (at 55.88 203.581 0))
+    (property "Value" "74LS04" (id 1) (at 57.912 199.517 0))
+    (property "Footprint" "Package_DIP:DIP-14_W7.62mm_Socket_LongPads" (id 2) (at 57.15 203.835 0)
+      (effects (font (size 1.27 1.27)) hide)
+    )
+    (property "Datasheet" "http://www.ti.com/lit/gpn/sn74LS04" (id 3) (at 57.15 203.835 0)
+      (effects (font (size 1.27 1.27)) hide)
+    )
+    (pin "1")
+    (pin "2")
+    (pin "3")
+    (pin "4")
+    (pin "5")
+    (pin "6")
+    (pin "8")
+    (pin "9")
+    (pin "10")
+    (pin "11")
+    (pin "12")
+    (pin "13")
+    (pin "14")
+    (pin "7")
+  )
   (symbol (lib_id "74xx:74LS74") (at 79.756 177.038 0) (mirror x) (unit 2)
     (in_bom yes) (on_board yes)
@@
     (pin "2")
   )
+  (symbol (lib_id "74xx:74LS14") (at 57.15 216.535 0) (unit 2)
+    (in_bom yes) (on_board yes)
+    (property "Reference" "U7" (id 0) (at 57.15 211.455 0))
+    (property "Value" "74LS14" (id 1) (at 56.515 212.725 0))
+    (property "Footprint" "Package_DIP:DIP-14_W7.62mm_Socket_LongPads" (id 2) (at 57.15 216.535 0)
+      (effects (font (size 1.27 1.27)) hide)
+    )
+    (property "Datasheet" "http://www.ti.com/lit/gpn/sn74LS14" (id 3) (at 57.15 216.535 0)
+      (effects (font (size 1.27 1.27)) hide)
+    )
+    (pin "1")
+    (pin "2")
+    (pin "3")
+    (pin "4")
+    (pin "5")
+    (pin "6")
+    (pin "8")
+    (pin "9")
+    (pin "10")
+    (pin "11")
+    (pin "12")
+    (pin "13")
+    (pin "14")
+    (pin "7")
+  )
   (symbol (lib_id "74xx:74LS08") (at 57.658 177.038 0) (unit 1)
