File: 22 processor.6502/hardware/processor.6502.kicad_pcb (KiCad board)
At the start: 2 copper layers, 235 x 160 mm, 116 parts, among them J1 IO Address Select, J11 FPANEL, J2 6809 RESET, J3 6809 ONLY, J4 RES SEL, J5 NMI Selection, J6 IRQ Selection, J7 I2C IRQ Selection, J8 UART IRQ Selection, P1 CONN_02X25, P2 CONN_02X25, P3 CONN_02X25, SW1 RESET, U1 74LS04, U10 74LS244, U11 74LS245, U12 74LS688, U13 CPU CLOCK, U14 74LS244, U15 DS1233, U16 74LS08, U17 74LS244, U18 UART CLOCK, U19 74LS157, U2 GAL16V8, U20 TL16C550CFN, U21 74LS74, U22 74LS688, U23 W65C02SxPL, U24 74LS670, U27 PCF8584, U29 74LS670, U3 GAL22V10, U31 74LS244, U33 74LS374, U4 74LS07, U5 27C010, U6 74LS244, U7 74LS14, U8 74LS244, U9 GAL22V10

Commit message: duodyne 6502 work
Parts:
- removed D1, D8: LED, LED_THT:LED_D3.0mm_Horizontal_O3.81mm_Z2.0mm
- removed R10, R6: 470, Resistor_THT:R_Axial_DIN0207_L6.3mm_D2.5mm_P7.62mm_Horizontal
- removed R11: 1K, Resistor_THT:R_Axial_DIN0207_L6.3mm_D2.5mm_P7.62mm_Horizontal
- J2: value 6809 RESET -> 6502 RESET
- J3: value 6809 ONLY -> 6502 ONLY
- U23: value W65C02SxPL -> 6502; footprint Package_LCC:PLCC-44_THT-Socket -> Package_DIP:DIP-40_W15.24mm_Socket_LongPads
- U5: value 27C010 -> 27C64; footprint Package_DIP:DIP-32_W15.24mm_Socket_LongPads -> Package_DIP:DIP-28_W15.24mm
- moved U23 19.4 mm to (93.4, 170.1), turned to 90 degrees
- moved R1 9.32 mm to (90.0, 95.4)
- moved C23 5.00 mm to (85.0, 165.0)
Connections:
- U1 pad 3: VP -> unconnected-(U1-Pad3)
- U1 pad 4: Net-(D8-Pad2) -> unconnected-(U1-Pad4)
- U23 pad 10: CPU-A0 -> CPU-A1
- U23 pad 11: CPU-A1 -> CPU-A2
- U23 pad 12: unconnected-(U23-Pad12) -> CPU-A3
- U23 pad 13: CPU-A2 -> CPU-A4
- U23 pad 14: CPU-A3 -> CPU-A5
- U23 pad 15: CPU-A4 -> CPU-A6
- U23 pad 16: CPU-A5 -> CPU-A7
- U23 pad 17: CPU-A6 -> CPU-A8
- U23 pad 18: CPU-A7 -> CPU-A9
- U23 pad 19: CPU-A8 -> CPU-A10
- U23 pad 2: VP -> ~{CPU-WAIT}
- U23 pad 20: CPU-A9 -> CPU-A11
- U23 pad 21: CPU-A10 -> GND
- U23 pad 22: CPU-A11 -> CPU-A12
- U23 pad 23: GND -> CPU-A13
- U23 pad 24: GND -> CPU-A14
- U23 pad 25: CPU-A12 -> CPU-A15
- U23 pad 26: CPU-A13 -> CPU-D7
- U23 pad 27: CPU-A14 -> CPU-D6
- U23 pad 28: CPU-A15 -> CPU-D5
- U23 pad 29: CPU-D7 -> CPU-D4
- U23 pad 3: ~{CPU-WAIT} -> unconnected-(U23-Pad3)
- U23 pad 30: CPU-D6 -> CPU-D3
- U23 pad 31: CPU-D5 -> CPU-D2
- U23 pad 32: CPU-D4 -> CPU-D1
- U23 pad 33: CPU-D3 -> CPU-D0
- U23 pad 34: CPU-D2 -> CPU-R~{W}
- U23 pad 35: CPU-D1 -> unconnected-(U23-Pad35)
- U23 pad 36: CPU-D0 -> unconnected-(U23-Pad36)
- U23 pad 37: VCC -> CLK
- U23 pad 38: CPU-R~{W} -> unconnected-(U23-Pad38)
- U23 pad 4: unconnected-(U23-Pad4) -> ~{CPU-INT}
- U23 pad 40: Net-(R11-Pad1) -> 6502RST
- U23 pad 5: ~{CPU-INT} -> unconnected-(U23-Pad5)
- U23 pad 6: ML -> ~{CPU-NMI}
- U23 pad 7: ~{CPU-NMI} -> SYNC
- U23 pad 8: SYNC -> VCC
- U23 pad 9: VCC -> CPU-A0
- U5 pad 10: CPU-A2 -> CPU-A0
- U5 pad 11: CPU-A1 -> CPU-D0
- U5 pad 12: CPU-A0 -> CPU-D1
- U5 pad 13: CPU-D0 -> CPU-D2
- U5 pad 14: CPU-D1 -> GND
- U5 pad 15: CPU-D2 -> CPU-D3
- U5 pad 16: GND -> CPU-D4
- U5 pad 17: CPU-D3 -> CPU-D5
- U5 pad 18: CPU-D4 -> CPU-D6
- U5 pad 19: CPU-D5 -> CPU-D7
- U5 pad 2: ZERO -> CPU-A12
- U5 pad 20: CPU-D6 -> ~{ONBOARD_ROM}
- U5 pad 21: CPU-D7 -> CPU-A10
- U5 pad 22: ~{ONBOARD_ROM} -> ZERO
- U5 pad 23: CPU-A10 -> CPU-A11
- U5 pad 24: ZERO -> CPU-A9
- U5 pad 25: CPU-A11 -> CPU-A8
- U5 pad 26: CPU-A9 -> unconnected-(U5-Pad26)
- U5 pad 27: CPU-A8 -> ONE
- U5 pad 28: ZERO -> unconnected-(U5-Pad28)
- U5 pad 3: ZERO -> CPU-A7
- U5 pad 4: CPU-A12 -> CPU-A6
- U5 pad 5: CPU-A7 -> CPU-A5
- U5 pad 6: CPU-A6 -> CPU-A4
- U5 pad 7: CPU-A5 -> CPU-A3
- U5 pad 8: CPU-A4 -> CPU-A2
- U5 pad 9: CPU-A3 -> CPU-A1
- U7 pad 3: ML -> unconnected-(U7-Pad3)
- U7 pad 4: Net-(D1-Pad2) -> unconnected-(U7-Pad4)
Routing:
- net GND: track 0.00 -> 1506.7 mm
- net VCC: track 0.00 -> 1178.9 mm
- net ~{RES_OUT}: track 0.00 -> 451.9 mm, vias 0 -> 3
- net ~{6502EN}: track 0.00 -> 433.8 mm, vias 0 -> 3
- net CPU-D4: track 0.00 -> 419.2 mm, vias 0 -> 3
- net CPU-D0: track 0.00 -> 412.0 mm, vias 0 -> 4
- net CPU-D6: track 0.00 -> 407.0 mm, vias 0 -> 3
- net ~{EIRQ0}: track 0.00 -> 400.0 mm, vias 0 -> 1
- net CPU-D5: track 0.00 -> 390.9 mm, vias 0 -> 3
- net ~{EIRQ4}: track 0.00 -> 386.7 mm
- net CPU-D7: track 0.00 -> 381.1 mm, vias 0 -> 5
- net CPU-D3: track 0.00 -> 379.4 mm, vias 0 -> 3
- net CPU-D1: track 0.00 -> 369.4 mm, vias 0 -> 3
- net CPU-D2: track 0.00 -> 367.1 mm, vias 0 -> 3
- net ~{EIRQ1}: track 0.00 -> 363.9 mm, vias 0 -> 1
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- added copper zone on B.Cu, net GND
- added copper zone on F.Cu, net GND
Other:
- board text added: "$9F"
- board text added: "6502 EN"
- board text added: "PROCESSOR.6502, VERSION 0.9, AS OF 26 APR 2025"
- board text removed: "$96"
- board text removed: "6809 EN"
- board text removed: "ML"
- board text removed: "PROCESSOR.6502, VERSION 0.8, AS OF 12 APR 2025"
- board text removed: "VP"
